File: PCB/rev3.0/1337-v3.0.kicad_sch (KiCad schematic)
At the start: 87 parts, among them J1 USB_IN, J2 AVR-ISP-6, J3 USB_OUT, Q1 FDS9926A, SW1 SW_Push, SW2 EC11, U1 CY7C65634-28LTXCT (or CY7C656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, U2 USBLC6-2SC6, U3 ATMEGA32U4, U4 USBLC6-2SC6, U5 SSD1306, Y1 12MHz, Y2 16MHz

Commit message: v3.0
Parts:
- SW2: footprint Rotary_Encoder:RotaryEncoder_Alps_EC11E-Switch_Vertical_H20mm_CircularMountingHoles -> 0xcb:RotaryEncoder_Alps_EC11E
Connections:
- net GND: now also J3.A1 (GND), J3.A12 (GND), J3.B1 (GND), J3.B12 (GND), J3.S1 (SHIELD), SW2.S1; no longer SW2.S2
- net S3: now also SW2.S2; no longer SW2.S1
- net VBUS1: now reaches C21.1, F2.1, J3.A4 (VBUS), J3.A9 (VBUS), J3.B4 (VBUS), J3.B9 (VBUS), U4.5 (VBUS)
- net VBUS: now reaches C6.1, F1.1, J1.A4 (VBUS), J1.A9 (VBUS), J1.B4 (VBUS), J1.B9 (VBUS), U2.5 (VBUS)
- net D-: now reaches U1.1 (0D-), U2.6 (IO1)
- net D+: now reaches U1.2 (0D+), U2.4 (IO2)
- net MCU+: now reaches R5.1, U3.4 (D+)
- net MCU-: now reaches R6.1, U3.3 (D-)
Other:
- moved on the sheet: R5, R6
Changed lines of the file:
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@@
   )
   (junction (at 25.4 63.5) (diameter 0.9144) (color 0 0 0 0))
+  (junction (at 26.035 115.57) (diameter 0.9144) (color 0 0 0 0))
   (junction (at 29.21 180.34) (diameter 0.9144) (color 0 0 0 0))
   (junction (at 29.845 154.305) (diameter 0.9144) (color 0 0 0 0))
@@
   (junction (at 58.42 154.305) (diameter 0.9144) (color 0 0 0 0))
   (junction (at 58.42 167.64) (diameter 0.9144) (color 0 0 0 0))
-  (junction (at 59.69 19.05) (diameter 0.9144) (color 0 0 0 0))
   (junction (at 69.85 17.78) (diameter 0.9144) (color 0 0 0 0))
   (junction (at 69.85 24.13) (diameter 0.9144) (color 0 0 0 0))
@@
     (stroke (width 0) (type solid) (color 0 0 0 0))
   )
-  (wire (pts (xy 88.265 173.355) (xy 105.41 173.355))
+  (wire (pts (xy 88.265 173.355) (xy 111.76 173.355))
     (stroke (width 0) (type solid) (color 0 0 0 0))
   )
@@
     (stroke (width 0) (type solid) (color 0 0 0 0))
   )
-  (wire (pts (xy 105.41 165.735) (xy 105.41 173.355))
-    (stroke (width 0) (type solid) (color 0 0 0 0))
-  )
   (wire (pts (xy 106.68 59.69) (xy 109.22 59.69))
     (stroke (width 0) (type solid) (color 0 0 0 0))
@@
     (stroke (width 0) (type solid) (color 0 0 0 0))
   )
+  (wire (pts (xy 111.76 160.655) (xy 105.41 160.655))
+    (stroke (width 0) (type solid) (color 0 0 0 0))
+  )
+  (wire (pts (xy 111.76 173.355) (xy 111.76 160.655))
+    (stroke (width 0) (type solid) (color 0 0 0 0))
+  )
   (wire (pts (xy 112.395 45.72) (xy 102.87 45.72))
     (stroke (width 0) (type solid) (color 0 0 0 0))
@@
     (stroke (width 0) (type solid) (color 0 0 0 0))
   )
-  (wire (pts (xy 224.155 43.815) (xy 225.425 43.815))
+  (wire (pts (xy 224.155 43.815) (xy 224.79 43.815))
     (stroke (width 0) (type solid) (color 0 0 0 0))
   )
-  (wire (pts (xy 224.155 46.355) (xy 225.425 46.355))
+  (wire (pts (xy 224.155 46.355) (xy 224.79 46.355))
     (stroke (width 0) (type solid) (color 0 0 0 0))
   )
@@
     (stroke (width 0) (type solid) (color 0 0 0 0))
   )
+  (wire (pts (xy 232.41 43.815) (xy 233.045 43.815))
+    (stroke (width 0) (type solid) (color 0 0 0 0))
+  )
+  (wire (pts (xy 232.41 46.355) (xy 233.045 46.355))
+    (stroke (width 0) (type solid) (color 0 0 0 0))
+  )
   (wire (pts (xy 233.045 23.495) (xy 233.045 24.765))
     (stroke (width 0) (type solid) (color 0 0 0 0))
@@
     (effects (font (size 5 5) (thickness 1) bold) (justify right bottom))
   )
+  (label "VBUS1" (at 45.72 71.12 180)
+    (effects (font (size 1.27 1.27)) (justify right bottom))
+  )
+  (label "VBUS" (at 46.355 25.4 180)
+    (effects (font (size 1.27 1.27)) (justify right bottom))
+  )
+  (label "D-" (at 78.74 40.64 180)
+    (effects (font (size 1.27 1.27)) (justify right bottom))
+  )
+  (label "D+" (at 78.74 43.18 180)
+    (effects (font (size 1.27 1.27)) (justify right bottom))
+  )
+  (label "MCU+" (at 233.045 43.815 0)
+    (effects (font (size 1.27 1.27)) (justify left bottom))
+  )
+  (label "MCU-" (at 233.045 46.355 0)
+    (effects (font (size 1.27 1.27)) (justify left bottom))
+  )
   (global_label "S1" (shape input) (at 20.955 137.16 180) (fields_autoplaced)
     (effects (font (size 1.27 1.27)) (justify right))
@@
     )
   )
-  (global_label "S3" (shape input) (at 105.41 160.655 0) (fields_autoplaced)
+  (global_label "S3" (shape input) (at 105.41 165.735 0) (fields_autoplaced)
     (effects (font (size 1.27 1.27)) (justify left))
-    (property "Intersheet References" "${INTERSHEET_REFS}" (id 0) (at 110.2421 160.5756 0)
+    (property "Intersheet References" "${INTERSHEET_REFS}" (id 0) (at 110.2421 165.6556 0)
       (effects (font (size 1.27 1.27)) (justify left) hide)
     )
@@
     (pin "1")
   )
+  (symbol (lib_id "power:GND") (at 26.035 115.57 0) (unit 1)
+    (in_bom yes) (on_board yes)
+    (property "Reference" "#PWR0102" (id 0) (at 26.035 121.92 0)
+      (effects (font (size 1.27 1.27)) hide)
+    )
+    (property "Value" "GND" (id 1) (at 26.035 120.015 0))
+    (property "Footprint" "" (id 2) (at 26.035 115.57 0)
+      (effects (font (size 1.27 1.27)) hide)
+    )
+    (property "Datasheet" "" (id 3) (at 26.035 115.57 0)
+      (effects (font (size 1.27 1.27)) hide)
+    )
+    (pin "1")
+  )
   (symbol (lib_id "power:GND") (at 26.035 142.24 0) (unit 1)
     (in_bom yes) (on_board yes)
@@
     (pin "2")
   )
-  (symbol (lib_id "Device:R") (at 229.235 43.815 270) (unit 1)
+  (symbol (lib_id "Device:R") (at 228.6 43.815 270) (unit 1)
     (in_bom yes) (on_board yes)
-    (property "Reference" "R5" (id 0) (at 225.425 42.545 90))
-    (property "Value" "22" (id 1) (at 229.235 43.815 90))
-    (property "Footprint" "Resistor_SMD:R_0603_1608Metric" (id 2) (at 229.235 42.037 90)
+    (property "Reference" "R5" (id 0) (at 224.79 42.545 90))
+    (property "Value" "22" (id 1) (at 228.6 43.815 90))
+    (property "Footprint" "Resistor_SMD:R_0603_1608Metric" (id 2) (at 228.6 42.037 90)
       (effects (font (size 1.27 1.27)) hide)
     )
-    (property "Datasheet" "~" (id 3) (at 229.235 43.815 0)
+    (property "Datasheet" "~" (id 3) (at 228.6 43.815 0)
       (effects (font (size 1.27 1.27)) hide)
     )
@@
     (pin "2")
   )
-  (symbol (lib_id "Device:R") (at 229.235 46.355 270) (unit 1)
+  (symbol (lib_id "Device:R") (at 228.6 46.355 270) (unit 1)
     (in_bom yes) (on_board yes)
-    (property "Reference" "R6" (id 0) (at 225.425 45.085 90))
-    (property "Value" "22" (id 1) (at 229.235 46.355 90))
-    (property "Footprint" "Resistor_SMD:R_0603_1608Metric" (id 2) (at 229.235 44.577 90)
+    (property "Reference" "R6" (id 0) (at 224.79 45.085 90))
+    (property "Value" "22" (id 1) (at 228.6 46.355 90))
+    (property "Footprint" "Resistor_SMD:R_0603_1608Metric" (id 2) (at 228.6 44.577 90)
       (effects (font (size 1.27 1.27)) hide)
     )
-    (property "Datasheet" "~" (id 3) (at 229.235 46.355 0)
+    (property "Datasheet" "~" (id 3) (at 228.6 46.355 0)
       (effects (font (size 1.27 1.27)) hide)
     )
@@
   (symbol (lib_id "Device:RotaryEncoder_Switch") (at 97.79 163.195 0) (unit 1)
     (in_bom yes) (on_board yes) (fields_autoplaced)
-    (property "Reference" "SW2" (id 0) (at 97.79 154.305 0))
-    (property "Value" "EC11" (id 1) (at 97.79 156.845 0))
-    (property "Footprint" "Rotary_Encoder:RotaryEncoder_Alps_EC11E-Switch_Vertical_H20mm_CircularMountingHoles" (id 2) (at 93.98 159.131 0)
+    (property "Reference" "SW2" (id 0) (at 97.79 153.67 0))
+    (property "Value" "EC11" (id 1) (at 97.79 156.21 0))
+    (property "Footprint" "0xcb:RotaryEncoder_Alps_EC11E" (id 2) (at 93.98 159.131 0)
       (effects (font (size 1.27 1.27)) hide)
     )
@@
       (reference "#PWR0101") (unit 1) (value "VCC") (footprint "")
     )
+    (path "/8ab124d8-9a09-473d-a4dd-0444cac1659b"
+      (reference "#PWR0102") (unit 1) (value "GND") (footprint "")
+    )
     (path "/31828b12-bfdc-463d-9d51-d301dcc63b5f"
       (reference "C1") (unit 1) (value "100n") (footprint "Capacitor_SMD:C_0603_1608Metric")
@@
     )
     (path "/b452cb47-3137-484b-8537-fda84715dce9"
-      (reference "SW2") (unit 1) (value "EC11") (footprint "Rotary_Encoder:RotaryEncoder_Alps_EC11E-Switch_Vertical_H20mm_CircularMountingHoles")
+      (reference "SW2") (unit 1) (value "EC11") (footprint "0xcb:RotaryEncoder_Alps_EC11E")
     )
     (path "/7d8f307a-1659-4dd1-8ebe-f7d96f0cbae3"
