File: PCB/rev3.0/1337-v3.0.kicad_sch (KiCad schematic)
At the start: 87 parts, among them J1 USB_IN, J2 AVR-ISP-6, J3 USB_OUT, Q1 FDS9926A, SW1 SW_Push, SW2 EC11, U1 CY7C65634-28LTXCT (or CY7C656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, U2 USBLC6-2SC6, U3 ATMEGA32U4, U4 USBLC6-2SC6, U5 SSD1306, Y1 12MHz, Y2 16MHz

Commit message: v3-proto
Parts:
- removed R1, R10, R24, R25, R26, R27, R4, R8: 10k, Resistor_SMD:R_0603_1608Metric, symbol Device:R
- added JP1, JP2: Jumper_2_Open, Resistor_SMD:R_0201_0603Metric, symbol Jumper:Jumper_2_Open
- added L1: LOGO, 0xcb:logo, symbol 0xcb:LOGO
- added L2: OSHW, 0xcb:oshw, symbol 0xcb:OSHW
- added RN1, RN2: 10k, Resistor_SMD:R_Array_Convex_4x0603, symbol Device:R_Pack04_Split
- C1, C10, C13, C14, C2, C21, C22, C23, C24, C25, C26, C27, C3, C6, C7, C8, C9: Alt Part Nb. (none) -> C91183; Part Nb. (none) -> 478-5266-1-ND
- C11, C12, C20, C4, C5: Alt Part Nb. (none) -> C393692; Part Nb. (none) -> 1276-1102-1-ND
- C15: Alt Part Nb. (none) -> C441753; Part Nb. (none) -> 587-3383-1-ND
- C16, C17, C18, C19: Alt Part Nb. (none) -> C85969; Part Nb. (none) -> 478-1167-1-ND
- D1, D2, D3, D4: Alt Part Nb. (none) -> C114586; Another Part Nb. (none) -> -; Part Nb. (none) -> 1568-COM-16347CT-ND
- F1: Alt Part Nb. (none) -> C369150; Part Nb. (none) -> 507-1815-1-ND
- F2: Alt Part Nb. (none) -> C883103; Part Nb. (none) -> 507-1813-1-ND
- FB1, FB2, FB3: Alt Part Nb. (none) -> C74330; Part Nb. (none) -> 732-1593-1-ND
- J1, J3: Alt Part Nb. (none) -> C223906; Another Part Nb. (none) -> -; Part Nb. (none) -> 900-2169900002CT-ND
- J2, U5: Alt Part Nb. (none) -> -; Another Part Nb. (none) -> -; Part Nb. (none) -> -; now left out of the parts list
- MX1, MX2, MX3, MX4, MX5, MX6, MX7, MX8, MX9: Alt Part Nb. (none) -> -; Another Part Nb. (none) -> -; Part Nb. (none) -> CH310-ND; now left out of the parts list
- Q1: Alt Part Nb. (none) -> C693202; Part Nb. (none) -> FDS9926ACT-ND
- R11, R12, R14, R28, R7, R9: Alt Part Nb. (none) -> C25804; Part Nb. (none) -> RHM10KADCT-ND
- R13: Alt Part Nb. (none) -> C705928; Part Nb. (none) -> P649DBCT-ND
- R15, R16, R17, R18, R19, R20, R21, R22, R23, R29: Alt Part Nb. (none) -> C104763; Part Nb. (none) -> A130532CT-ND
- R2, R3: Alt Part Nb. (none) -> C23186; Part Nb. (none) -> P5.1KDBCT-ND
- R5, R6: Alt Part Nb. (none) -> C174301; Part Nb. (none) -> A130081CT-ND
- SW1: Alt Part Nb. (none) -> C318884; Part Nb. (none) -> EG2531CT-ND
- SW2: Alt Part Nb. (none) -> C278348; Another Part Nb. (none) -> -; Part Nb. (none) -> PEC11L-4125F-S0020-ND; now left out of the parts list
- U1: Alt Part Nb. (none) -> C1521581; Another Part Nb. (none) -> https://www.win-source.net/cypress-semiconductor-corp-cy7c6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; Part Nb. (none) -> 428-3154-1-ND
- U2, U4: Alt Part Nb. (none) -> C7519; Part Nb. (none) -> 497-5235-1-ND
- U3: Alt Part Nb. (none) -> C112161; Part Nb. (none) -> ATMEGA32U4RC-MURCT-ND
- Y1: Alt Part Nb. (none) -> C9002; Part Nb. (none) -> XC2874CT-ND
- Y2: Alt Part Nb. (none) -> C389842; Part Nb. (none) -> XC2060CT-ND
Connections:
- net +3V3: now also RN1.1 (R1.1), RN1.2 (R2.1), RN1.3 (R3.1), RN1.4 (R4.1)
- net 1D+: now also JP2.1 (A)
- net 1D-: now also JP1.1 (A)
- net D+: now also JP2.2 (B)
- net D-: now also JP1.2 (B)
- net EA: now also RN2.7 (R2.2)
- net EB: now also RN2.6 (R3.2)
- net VCC: now also RN2.1 (R1.1), RN2.4 (R4.1)
- net at U1.25 (OVR1): now also RN1.8 (R1.2)
- net at U1.19 (OVR4): now also RN1.6 (R3.2)
- net at U1.24 (OVR2): now also RN1.7 (R2.2)
- net at U1.20 (OVR3): now also RN1.5 (R4.2)
- net at SW2.B: now also RN2.3 (R3.1), RN2.5 (R4.2)
- net at SW2.A: now also RN2.2 (R2.1), RN2.8 (R1.2)

Commit message: update bom
Parts:
- JP1, JP2: now left out of the parts list
- RN1, RN2: Alt Part Nb. (none) -> C109324; Part Nb. (none) -> MNR14103RTR-ND
Changed lines of the file:
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@@
+      (effects (font (size 1.27 1.27)) hide)
+    )
+    (property "Alt Part Nb." "C109324" (id 4) (at 81.28 160.655 0)
+      (effects (font (size 1.27 1.27)) hide)
+    )
+    (property "Part Nb." "MNR14103RTR-ND" (id 5) (at 81.28 160.655 0)
       (effects (font (size 1.27 1.27)) hide)
     )
@@
       (effects (font (size 1.27 1.27)) hide)
     )
+    (property "Alt Part Nb." "C109324" (id 4) (at 83.185 165.735 0)
+      (effects (font (size 1.27 1.27)) hide)
+    )
+    (property "Part Nb." "MNR14103RTR-ND" (id 5) (at 83.185 165.735 0)
+      (effects (font (size 1.27 1.27)) hide)
+    )
     (pin "3")
     (pin "6")
@@
       (effects (font (size 1.27 1.27)) hide)
     )
+    (property "Alt Part Nb." "C109324" (id 4) (at 85.09 154.94 0)
+      (effects (font (size 1.27 1.27)) hide)
+    )
+    (property "Part Nb." "MNR14103RTR-ND" (id 5) (at 85.09 154.94 0)
+      (effects (font (size 1.27 1.27)) hide)
+    )
     (pin "1")
     (pin "8")
@@
     )
     (property "Datasheet" "~" (id 3) (at 86.995 154.94 0)
+      (effects (font (size 1.27 1.27)) hide)
+    )
+    (property "Alt Part Nb." "C109324" (id 4) (at 86.995 154.94 0)
+      (effects (font (size 1.27 1.27)) hide)
+    )
+    (property "Part Nb." "MNR14103RTR-ND" (id 5) (at 86.995 154.94 0)
       (effects (font (size 1.27 1.27)) hide)
     )
@@
       (effects (font (size 1.27 1.27)) hide)
     )
+    (property "Alt Part Nb." "C109324" (id 4) (at 146.05 29.21 0)
+      (effects (font (size 1.27 1.27)) hide)
+    )
+    (property "Part Nb." "MNR14103RTR-ND" (id 5) (at 146.05 29.21 0)
+      (effects (font (size 1.27 1.27)) hide)
+    )
     (pin "1")
     (pin "8")
@@
       (effects (font (size 1.27 1.27)) hide)
     )
+    (property "Alt Part Nb." "C109324" (id 4) (at 146.05 39.37 0)
+      (effects (font (size 1.27 1.27)) hide)
+    )
+    (property "Part Nb." "MNR14103RTR-ND" (id 5) (at 146.05 39.37 0)
+      (effects (font (size 1.27 1.27)) hide)
+    )
     (pin "2")
     (pin "7")
@@
       (effects (font (size 1.27 1.27)) hide)
     )
+    (property "Alt Part Nb." "C109324" (id 4) (at 146.05 49.53 0)
+      (effects (font (size 1.27 1.27)) hide)
+    )
+    (property "Part Nb." "MNR14103RTR-ND" (id 5) (at 146.05 49.53 0)
+      (effects (font (size 1.27 1.27)) hide)
+    )
     (pin "4")
     (pin "5")
@@
       (effects (font (size 1.27 1.27)) hide)
     )
+    (property "Alt Part Nb." "C109324" (id 4) (at 146.05 59.69 0)
+      (effects (font (size 1.27 1.27)) hide)
+    )
+    (property "Part Nb." "MNR14103RTR-ND" (id 5) (at 146.05 59.69 0)
+      (effects (font (size 1.27 1.27)) hide)
+    )
     (pin "3")
     (pin "6")
@@
   )
   (symbol (lib_id "Jumper:Jumper_2_Open") (at 83.185 48.26 90) (unit 1)
-    (in_bom yes) (on_board yes)
+    (in_bom no) (on_board yes)
     (property "Reference" "JP2" (id 0) (at 81.915 48.2599 90)
       (effects (font (size 1.27 1.27)) (justify right))
@@
   )
   (symbol (lib_id "Jumper:Jumper_2_Open") (at 86.995 45.72 90) (unit 1)
-    (in_bom yes) (on_board yes)
+    (in_bom no) (on_board yes)
     (property "Reference" "JP1" (id 0) (at 85.725 45.7199 90)
       (effects (font (size 1.27 1.27)) (justify right))
