File: PCB/rev3.0/1337-v3.0.kicad_pcb (KiCad board)
At the start: 2 copper layers, 62 x 62 mm, 87 parts, among them J1 USB_IN, J2 AVR-ISP-6, J3 USB_OUT, Q1 FDS9926A, SW1 SW_Push, SW2 EC11, U1 CY7C65634-28LTXCT (or CY7C656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, U2 USBLC6-2SC6, U3 ATMEGA32U4, U4 USBLC6-2SC6, U5 SSD1306, Y1 12MHz, Y2 16MHz

Commit message: v3-proto
Parts:
- removed R1, R10, R24, R25, R26, R27, R4, R8: 10k, Resistor_SMD:R_0603_1608Metric
- added JP1: Jumper_2_Open, Resistor_SMD:R_0201_0603Metric, B.Cu at (162.7, 84.0)
- added JP2: Jumper_2_Open, Resistor_SMD:R_0201_0603Metric, B.Cu at (164.7, 84.0)
- added L***: oshwa, 0xcb:oshwa, B.Cu at (154.9, 128.1)
- added L1: LOGO, 0xcb:logo, B.Cu at (139.3, 97.6)
- added L2: OSHW, 0xcb:oshw, B.Cu at (173.7, 110.2)
- added RN1: 10k, Resistor_SMD:R_Array_Convex_4x0603, B.Cu at (151.5, 92.5)
- added RN2: 10k, Resistor_SMD:R_Array_Convex_4x0603, B.Cu at (174.2, 92.4)
- moved R6 9.86 mm to (162.7, 86.1)
- moved R5 9.00 mm to (164.7, 86.1)
- moved R11 3.06 mm to (154.2, 92.4)
- moved R9 2.33 mm to (148.9, 92.5)
- moved FB1 1.70 mm to (158.5, 85.1), turned to 180 degrees
- moved C20 1.56 mm to (167.4, 115.6), turned to 0 degrees
- moved MX6 0.10 mm to (173.9, 100.7)
- moved MX5 0.10 mm to (148.7, 100.7)
- moved MX3 0.08 mm to (174.0, 81.6)
- moved MX1 0.08 mm to (129.8, 81.6)
- moved MX2 0.08 mm to (148.8, 81.6)
- moved MX4 0.08 mm to (129.8, 100.6)
- moved MX7 0.08 mm to (129.8, 119.7)
- moved MX8 0.08 mm to (148.8, 119.7)
- moved MX9 0.08 mm to (174.0, 119.7)
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Routing:
- net VCC: track 310.2 -> 295.0 mm, vias 8 -> 10
- net /MCU-: track 25.5 -> 34.2 mm
- net /MCU+: track 26.3 -> 33.8 mm, vias 2 -> 0
- net 2D-: track 30.1 -> 35.8 mm
- net 2D+: track 29.0 -> 34.2 mm
- net Net-(D3-Pad2): track 17.9 -> 22.8 mm, vias 0 -> 2
- net Net-(RN1-Pad6): track 10.6 -> 5.88 mm
- net Net-(RN1-Pad7): track 2.79 -> 6.08 mm
- net Net-(R11-Pad2): track 4.82 -> 1.76 mm
- net 1D+: track 9.10 -> 12.1 mm
- net Net-(D2-Pad2): track 31.9 -> 29.0 mm
- net Net-(RN1-Pad5): track 7.56 -> 4.73 mm
- net Net-(R9-Pad2): track 12.7 -> 9.97 mm
- net Net-(RN1-Pad8): track 4.64 -> 7.30 mm
- net EA: track 34.2 -> 36.0 mm
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Other:
- board text added: "USB JMP"
- board text added: "https://0xCB.dev"
