File: rev5.0/pcb.kicad_pcb (KiCad board)
At the start: 4 copper layers, 62 x 62 mm, 121 parts, among them J1 USB_C_Receptacle_USB2.0, J2 FPC, J3 J-LINK_6-PIN_NEEDLE_ADAPTER, U1 USBLC6-2P6, U2 XC6210B332MR-G, U3 TPS2553DBVR, U4 74LVC1T45, U5 W25Q32JVUUIQ, U6 RP2040, Y1 12MHz

Commit message: prod file generation
Parts:
- D1, D2, D3, D4, D5, D6, D7, D8, MX1, MX2, MX4, MX5, MX6, MX7, MX8, MX9: moved to B.Cu
- R6: value 1K -> 1k
- turned D1 to 180 degrees
- turned D2 to 180 degrees
- turned D3 to 180 degrees
- turned D4 to 180 degrees
- turned D5 to 180 degrees
- turned D6 to 180 degrees
- turned D7 to 180 degrees
- turned D8 to 180 degrees
- turned MX1 to 180 degrees
- turned MX2 to 180 degrees
- turned MX4 to 180 degrees
- turned MX5 to 180 degrees
- turned MX6 to 180 degrees
- turned MX7 to 180 degrees
- turned MX8 to 180 degrees
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