File: rev5.0/pcb.kicad_sch (KiCad schematic)
At the start: 115 parts, among them J2 FPC, U3 TPS2553DBVR, U3 XC6210B332MR-G

Commit message: prod file generation
Parts:
- D1, D2, D3, D4, D5, D6, D7, D8: JLCPCB_CORRECTION (none) -> 0; -3; 180
- D? (x11): JLCPCB_CORRECTION (none) -> 0; 0; 180; LCSC C965555 -> C2976072
- D? (x12): JLCPCB_CORRECTION (none) -> 0; 0; 0; LCSC C965555 -> C2976072
- FB? (x2): LCSC C88960 -> C160977
- J2: JLCPCB_CORRECTION (none) -> 0; 3; 180
- J?: JLCPCB_CORRECTION (none) -> 0; 1.5; 180
- MX1, MX2, MX4, MX5, MX6, MX7, MX8, MX9: JLCPCB_CORRECTION (none) -> 0.2; 3.5; 0
- MX3: JLCPCB_CORRECTION (none) -> -6; 2; 270; now in the parts list
- R? (x2): LCSC C11702 -> C138165
- RN1, U?: JLCPCB_CORRECTION (none) -> 0; 0; 90
- U3, U?: JLCPCB_CORRECTION (none) -> 0; 0; 180

Commit message: fix some minor issues
Parts:
- C? (x2): LCSC C237458 -> C76935
- MX3: Alt Part Nb. C278348 -> C143788
- R?: value 75k -> 40k; LCSC C25744 -> C274875
- R? (x2): LCSC C138165 -> C138297
Changed lines of the file:
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@@
       (effects (font (size 1.27 1.27)) hide)
     )
-    (property "LCSC" "C237458" (at 283.21 116.84 0)
+    (property "LCSC" "C76935" (at 283.21 116.84 0)
       (effects (font (size 1.27 1.27)) hide)
     )
@@
       (effects (font (size 1.27 1.27)) hide)
     )
-    (property "Alt Part Nb." "C278348" (at 101.6 139.7 0)
+    (property "Alt Part Nb." "C143788" (at 101.6 139.7 0)
       (effects (font (size 1.27 1.27)) hide)
     )
@@
       (effects (font (size 1.27 1.27)) hide)
     )
-    (property "LCSC" "C237458" (at 283.21 111.76 0)
+    (property "LCSC" "C76935" (at 283.21 111.76 0)
       (effects (font (size 1.27 1.27)) hide)
     )
@@
       (effects (font (size 1.27 1.27)) (justify left))
     )
-    (property "Value" "75k" (at 154.94 80.01 0)
+    (property "Value" "40k" (at 154.94 80.01 0)
       (effects (font (size 1.27 1.27)) (justify left))
     )
@@
       (effects (font (size 1.27 1.27)) hide)
     )
-    (property "LCSC" "C25744" (at 160.02 78.74 0)
+    (property "LCSC" "C274875" (at 160.02 78.74 0)
       (effects (font (size 1.27 1.27)) hide)
     )
@@
       (effects (font (size 1.27 1.27)) hide)
     )
-    (property "LCSC" "C138165" (at 288.29 152.4 0)
+    (property "LCSC" "C138297" (at 288.29 152.4 0)
       (effects (font (size 1.27 1.27)) hide)
     )
@@
       (effects (font (size 1.27 1.27)) hide)
     )
-    (property "LCSC" "C138165" (at 353.06 87.63 0)
+    (property "LCSC" "C138297" (at 353.06 87.63 0)
       (effects (font (size 1.27 1.27)) hide)
     )
