File: rev5.0/flex-cable/Rev1.0/pcb.kicad_sch (KiCad schematic)
At the start: 2 parts, among them J1 fpc, J2 oled

Commit message: fix some minor issues
Connections:
- net GND: now also J1.11 (Pin_11), J1.12 (Pin_12); no longer J1.1 (Pin_1), J1.2 (Pin_2)
- net VCC: now also J1.1 (Pin_1), J1.2 (Pin_2); no longer J1.11 (Pin_11), J1.12 (Pin_12)
- net i2c_scl: now also J1.9 (Pin_9); no longer J1.4 (Pin_4)
- net i2c_sda: now also J1.10 (Pin_10); no longer J1.3 (Pin_3)
- net misc: now also J1.3 (Pin_3); no longer J1.10 (Pin_10)
- net spi_cs: now also J1.8 (Pin_8); no longer J1.5 (Pin_5)
- net spi_dc: now also J1.7 (Pin_7); no longer J1.6 (Pin_6)
- net spi_rst: now also J1.4 (Pin_4); no longer J1.9 (Pin_9)
- net spi_sdi: now also J1.5 (Pin_5); no longer J1.8 (Pin_8)
- net spi_sdo: now also J1.6 (Pin_6); no longer J1.7 (Pin_7)
Changed lines of the file:
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@@
-    )
-  )
-  (symbol (lib_id "Connector:Conn_01x12_Pin") (at 139.7 116.332 0) (unit 1)
-    (in_bom yes) (on_board yes) (dnp no) (fields_autoplaced)
-    (property "Reference" "J1" (at 140.335 99.06 0)
-      (effects (font (size 1.27 1.27)))
-    )
-    (property "Value" "fpc" (at 140.335 101.6 0)
-      (effects (font (size 1.27 1.27)))
-    )
-    (property "Footprint" "Library:FFC-SMD_12P-P0.50_X05B20U12T" (at 139.7 116.332 0)
-      (effects (font (size 1.27 1.27)) hide)
-    )
-    (property "Datasheet" "~" (at 139.7 116.332 0)
-      (effects (font (size 1.27 1.27)) hide)
-    )
-    (pin "1")
-    (pin "10")
-    (pin "11")
-    (pin "12")
-    (pin "2")
-    (pin "3")
-    (pin "4")
-    (pin "5")
-    (pin "6")
-    (pin "7")
-    (pin "8")
-    (pin "9")
-    (instances
-      (project "pcb"
-        (path "/59f16264-4fca-4d31-9679-edff70f988cd"
-          (reference "J1") (unit 1)
-        )
-      )
     )
   )
@@
         )
       )
+    )
+  )
+  (symbol (lib_id "Connector:Conn_01x12_Pin") (at 139.7 118.872 0) (mirror x) (unit 1)
+    (in_bom yes) (on_board yes) (dnp no)
+    (property "Reference" "J1" (at 140.335 136.144 0)
+      (effects (font (size 1.27 1.27)))
+    )
+    (property "Value" "fpc" (at 140.335 133.604 0)
+      (effects (font (size 1.27 1.27)))
+    )
+    (property "Footprint" "Library:FFC-SMD_12P-P0.50_X05B20U12T" (at 139.7 118.872 0)
+      (effects (font (size 1.27 1.27)) hide)
+    )
+    (property "Datasheet" "~" (at 139.7 118.872 0)
+      (effects (font (size 1.27 1.27)) hide)
+    )
+    (pin "1")
+    (pin "10")
+    (pin "11")
+    (pin "12")
+    (pin "2")
+    (pin "3")
+    (pin "4")
+    (pin "5")
+    (pin "6")
+    (pin "7")
+    (pin "8")
+    (pin "9")
+    (instances
+      (project "pcb"
+        (path "/59f16264-4fca-4d31-9679-edff70f988cd"
+          (reference "J1") (unit 1)
+        )
+      )
